Commit message: update robot model

File: udacity_bot/urdf/udacity_bot.xacro (robot description, xacro)
@@ -1,4 +1,5 @@
 <?xml version='1.0'?>
 <robot name="udacity_bot" xmlns:xacro="http://www.ros.org/wiki/xacro">
+  <xacro:include filename="$(find udacity_bot)/urdf/udacity_bot.gazebo" />
   <link name="robot_footprint"></link>
   <joint name="robot_footprint_joint" type="fixed">
@@ -139,3 +140,61 @@
     <joint_properties damping="1.0" friction="1.0"/>
   </joint>
+  <link name="camera">
+    <pose>0 0 0 0 0 0</pose>
+    <inertial>
+      <mass value="0.1"/>
+      <origin xyz="0 0 0" rpy=" 0 0 0"/>
+      <inertia
+          ixx="1e-6" ixy="0" ixz="0"
+          iyy="1e-6" iyz="0"
+          izz="1e-6"
+      />
+    </inertial>
+    <collision>
+      <origin xyz="0 0.025 0" rpy=" 1.57075 0 0"/>
+      <geometry>
+        <box size=".05 .05 .05"/>
+      </geometry>
+    </collision>
+    <visual>
+      <origin xyz="0 0.025 0" rpy=" 1.57075 0 0"/>
+      <geometry>
+        <box size=".05 .05 .05"/>
+      </geometry>
+    </visual>
+  </link>
+  <joint type="fixed" name="camera_joint">
+    <origin xyz="0.2 0 0" rpy="0 0 0"/>
+    <child link="camera"/>
+    <parent link="chassis"/>
+  </joint>
+  <link name="hokuyo">
+    <pose>0 0 0 0 0 0</pose>
+    <inertial>
+      <mass value="0.1"/>
+      <origin xyz="0 0 0" rpy=" 0 0 0"/>
+      <inertia
+          ixx="1e-6" ixy="0" ixz="0"
+          iyy="1e-6" iyz="0"
+          izz="1e-6"
+      />
+    </inertial>
+    <collision>
+      <origin xyz="0 0 0" rpy=" 0 0 0"/>
+      <geometry>
+        <box size=".1 .1 .1"/>
+      </geometry>
+    </collision>
+    <visual>
+      <origin xyz="0 0 0" rpy=" 0 0 0"/>
+      <geometry>
+        <mesh filename="package://udacity_bot/meshes/hokuyo.dae"/>
+      </geometry>
+    </visual>
+  </link>
+  <joint type="fixed" name="hokuyo_joint">
+    <origin xyz="0.15 0 0.1" rpy="0 0 0"/>
+    <child link="hokuyo"/>
+    <parent link="chassis"/>
+  </joint>
 </robot>

Commit message: update wheel

File: udacity_bot/urdf/udacity_bot.xacro (robot description, xacro)
@@ -77,5 +77,4 @@
   </link>
   <link name='left_wheel'>
-    <pose>0 0 0 0 1.5707 1.5707</pose>
     <inertial>
       <mass value="5.0"/>
@@ -88,5 +87,5 @@
     </inertial>
     <collision>
-      <origin xyz="0 -0.025 0" rpy=" 1.57075 0 0"/>
+      <origin xyz="0 0 0 0" rpy="0 1.5707 1.5707"/>
       <geometry>
         <cylinder radius="0.1" length="0.05"/>
@@ -94,5 +93,5 @@
     </collision>
     <visual>
-      <origin xyz="0 -0.025 0" rpy=" 1.57075 0 0"/>
+      <origin xyz="0 0 0 0" rpy="0 1.5707 1.5707"/>
       <geometry>
         <cylinder radius="0.1" length="0.05"/>

Commit message: update left wheel gazebo

File: udacity_bot/urdf/udacity_bot.xacro (robot description, xacro)
@@ -77,8 +77,7 @@
   </link>
   <link name='left_wheel'>
-    <pose>0 0 0 0 1.5707 1.5707</pose>
     <inertial>
       <mass value="5.0"/>
-      <origin xyz="0.0 0 0" rpy=" 0 0 0"/>
+      <origin xyz="0 0 0" rpy="0 1.5707 1.5707"/>
       <inertia
           ixx="0.1" ixy="0" ixz="0"
@@ -88,5 +87,5 @@
     </inertial>
     <collision>
-      <origin xyz="0 -0.025 0" rpy=" 1.57075 0 0"/>
+      <origin xyz="0 0 0" rpy="0 1.5707 1.5707"/>
       <geometry>
         <cylinder radius="0.1" length="0.05"/>
@@ -94,5 +93,5 @@
     </collision>
     <visual>
-      <origin xyz="0 -0.025 0" rpy=" 1.57075 0 0"/>
+      <origin xyz="0 0 0" rpy="0 1.5707 1.5707"/>
       <geometry>
         <cylinder radius="0.1" length="0.05"/>

Commit message: update right and left wheel

File: udacity_bot/urdf/udacity_bot.xacro (robot description, xacro)
@@ -77,7 +77,8 @@
   </link>
   <link name='left_wheel'>
+    <!--pose>0 0 0 0 1.5707 1.5707</pose-->
     <inertial>
       <mass value="5.0"/>
-      <origin xyz="0 0 0" rpy="0 1.5707 1.5707"/>
+      <origin xyz="0.0 0 0" rpy=" 0 0 0"/>
       <inertia
           ixx="0.1" ixy="0" ixz="0"
@@ -87,11 +88,13 @@
     </inertial>
     <collision>
-      <origin xyz="0 0 0" rpy="0 1.5707 1.5707"/>
-      <geometry>
-        <cylinder radius="0.1" length="0.05"/>
-      </geometry>
-    </collision>
-    <visual>
-      <origin xyz="0 0 0" rpy="0 1.5707 1.5707"/>
+      <!--origin xyz="0 -0.025 0" rpy=" 1.57075 0 0"/-->
+      <origin xyz="0 0 0" rpy=" 0 1.5707 1.5707"/>
+      <geometry>
+        <cylinder radius="0.1" length="0.05"/>
+      </geometry>
+    </collision>
+    <visual>
+      <!--origin xyz="0 -0.025 0" rpy=" 1.57075 0 0"/-->
+      <origin xyz="0 0 0" rpy=" 0 1.5707 1.5707"/>
       <geometry>
         <cylinder radius="0.1" length="0.05"/>
@@ -108,5 +111,5 @@
   </joint>
   <link name='right_wheel'>
-    <pose>0 0 0 0 1.5707 1.5707</pose>
+    <!--pose>0 0 0 0 1.5707 1.5707</pose-->
     <inertial>
       <mass value="5.0"/>
@@ -119,11 +122,13 @@
     </inertial>
     <collision>
-      <origin xyz="0 0.025 0" rpy=" 1.57075 0 0"/>
-      <geometry>
-        <cylinder radius="0.1" length="0.05"/>
-      </geometry>
-    </collision>
-    <visual>
-      <origin xyz="0 0.025 0" rpy=" 1.57075 0 0"/>
+      <!--origin xyz="0 0.025 0" rpy=" 1.57075 0 0"/-->
+      <origin xyz="0 0 0" rpy=" 0 1.5707 1.5707"/>
+      <geometry>
+        <cylinder radius="0.1" length="0.05"/>
+      </geometry>
+    </collision>
+    <visual>
+      <!--origin xyz="0 0.025 0" rpy=" 1.57075 0 0"/-->
+      <origin xyz="0 0 0" rpy=" 0 1.5707 1.5707"/>
       <geometry>
         <cylinder radius="0.1" length="0.05"/>

Commit message: @changes@

File: udacity_bot/urdf/udacity_bot.xacro (robot description, xacro)
@@ -87,5 +87,5 @@
     </inertial>
     <collision>
-      <origin xyz="0 -0.025 0" rpy=" 1.57075 0 0"/>
+      <origin xyz="0 0 0" rpy=" 0 1.5707 1.5707"/>
       <geometry>
         <cylinder radius="0.1" length="0.05"/>
@@ -93,5 +93,5 @@
     </collision>
     <visual>
-      <origin xyz="0 -0.025 0" rpy=" 1.57075 0 0"/>
+      <origin xyz="0 0 0" rpy=" 0 1.5707 1.5707"/>
       <geometry>
         <cylinder radius="0.1" length="0.05"/>
@@ -108,5 +108,4 @@
   </joint>
   <link name='right_wheel'>
-    <pose>0 0 0 0 1.5707 1.5707</pose>
     <inertial>
       <mass value="5.0"/>
@@ -119,5 +118,5 @@
     </inertial>
     <collision>
-      <origin xyz="0 0.025 0" rpy=" 1.57075 0 0"/>
+      <origin xyz="0 0 0" rpy=" 0 1.5707 1.5707"/>
       <geometry>
         <cylinder radius="0.1" length="0.05"/>
@@ -125,5 +124,5 @@
     </collision>
     <visual>
-      <origin xyz="0 0.025 0" rpy=" 1.57075 0 0"/>
+      <origin xyz="0 0 0" rpy=" 0 1.5707 1.5707"/>
       <geometry>
         <cylinder radius="0.1" length="0.05"/>

Commit message: update robot model with a new look

File: udacity_bot/urdf/udacity_bot.xacro (robot description, xacro)
@@ -2,4 +2,10 @@
 <robot name="udacity_bot" xmlns:xacro="http://www.ros.org/wiki/xacro">
   <xacro:include filename="$(find udacity_bot)/urdf/udacity_bot.gazebo" />
+  <material name="blue">
+    <color rgba="0.28 0.6 0.6 1"/>
+  </material>
+  <material name="light_blue">
+    <color rgba="0.28 0.6 0.9 0.8"/>
+  </material>
   <link name="robot_footprint"></link>
   <joint name="robot_footprint_joint" type="fixed">
@@ -22,5 +28,5 @@
       <origin xyz="0 0 0" rpy=" 0 0 0"/>
       <geometry>
-        <box size=".4 .2 .1"/>
+        <cylinder radius="0.2" length="0.1"/>
       </geometry>
     </collision>
@@ -28,6 +34,7 @@
       <origin xyz="0 0 0" rpy=" 0 0 0"/>
       <geometry>
-        <box size=".4 .2 .1"/>
-      </geometry>
+        <cylinder radius="0.2" length="0.1"/>
+      </geometry>
+      <material name="light_blue"/>
     </visual>
     <collision name='back_caster_collision'>
@@ -89,16 +96,17 @@
       <origin xyz="0 0 0" rpy=" 0 1.5707 1.5707"/>
       <geometry>
-        <cylinder radius="0.1" length="0.05"/>
-      </geometry>
-    </collision>
-    <visual>
-      <origin xyz="0 0 0" rpy=" 0 1.5707 1.5707"/>
-      <geometry>
-        <cylinder radius="0.1" length="0.05"/>
-      </geometry>
+        <cylinder radius="0.05" length="0.05"/>
+      </geometry>
+    </collision>
+    <visual>
+      <origin xyz="0 0 0" rpy=" 0 1.5707 1.5707"/>
+      <geometry>
+        <cylinder radius="0.05" length="0.05"/>
+      </geometry>
+      <material name="blue"/>
     </visual>
   </link>
   <joint type="continuous" name="left_wheel_hinge">
-    <origin xyz="0 0.15 0" rpy="0 0 0"/>
+    <origin xyz="0 0.15 -0.05" rpy="0 0 0"/>
     <child link="left_wheel"/>
     <parent link="chassis"/>
@@ -120,16 +128,17 @@
       <origin xyz="0 0 0" rpy=" 0 1.5707 1.5707"/>
       <geometry>
-        <cylinder radius="0.1" length="0.05"/>
-      </geometry>
-    </collision>
-    <visual>
-      <origin xyz="0 0 0" rpy=" 0 1.5707 1.5707"/>
-      <geometry>
-        <cylinder radius="0.1" length="0.05"/>
-      </geometry>
+        <cylinder radius="0.05" length="0.05"/>
+      </geometry>
+    </collision>
+    <visual>
+      <origin xyz="0 0 0" rpy=" 0 1.5707 1.5707"/>
+      <geometry>
+        <cylinder radius="0.05" length="0.05"/>
+      </geometry>
+      <material name="blue"/>
     </visual>
   </link>
   <joint type="continuous" name="right_wheel_hinge">
-    <origin xyz="0 -0.15 0" rpy="0 0 0"/>
+    <origin xyz="0 -0.15 -0.05" rpy="0 0 0"/>
     <child link="right_wheel"/>
     <parent link="chassis"/>
@@ -150,5 +159,5 @@
     </inertial>
     <collision>
-      <origin xyz="0 0.025 0" rpy=" 1.57075 0 0"/>
+      <origin xyz="0 0 0" rpy=" 1.57075 0 0"/>
       <geometry>
         <box size=".05 .05 .05"/>
@@ -156,5 +165,5 @@
     </collision>
     <visual>
-      <origin xyz="0 0.025 0" rpy=" 1.57075 0 0"/>
+      <origin xyz="0 0 0" rpy=" 1.57075 0 0"/>
       <geometry>
         <box size=".05 .05 .05"/>
